Commit message: Add gui to control robot, update launcher to publish to robot updates. URDF is fixed as matlab code and DH

File: src/quadruped_arm_motion/urdf/quadruped_arm.urdf (robot description, URDF)
Before this commit: robot quadruped_arm_robot, 33 links, 32 joints
Joints:
- joint backLeft_ankle_joint: origin xyz=0.25 -0.0000 0 rpy=0 0 -1.5708 -> xyz=0.25 -0.0000 0 rpy=0 0 0
- joint backLeft_hip_motor_joint: origin xyz=0 0 0 rpy=0 1.5708 1.5708 -> xyz=0 0 0 rpy=-1.5708  0 -1.5708
- joint backLeft_knee_joint: origin xyz=-0.05 0 0 rpy=1.5708 0.0000 0.7854 -> xyz=0.1 0 0 rpy=-1.5708 0.0000 0
- joint backRight_ankle_joint: origin xyz=0 0 0.25 rpy=0 0 -1.5708 -> xyz=0.25 0 0 rpy=0 0 0
- joint backRight_hip_motor_joint: origin xyz=0 0 0 rpy=0 -1.5708 -1.5708 -> xyz=0 0 0 rpy=1.5708  0 -1.5708
- joint backRight_knee_joint: origin xyz=0.05 0 0 rpy=1.5708 0.0000 0.7854 -> xyz=0.1 0 0 rpy=1.5708 0   0
- joint frontLeft_ankle_joint: origin xyz=0.25 -0.0000 0 rpy=0 0 -1.5708 -> xyz=0.25 -0.0000 0 rpy=0 0 0
- joint frontLeft_hip_motor_joint: origin xyz=0 0 0 rpy=0 1.5708 1.5708 -> xyz=0 0 0 rpy=-1.5708  0 -1.5708
- joint frontLeft_knee_joint: origin xyz=-0.05 0 0 rpy=1.5708 0.0000 0.7854 -> xyz=0.1 0 0 rpy=-1.5708 0.0000 0
- joint frontRight_ankle_joint: origin xyz=0 0 0.25 rpy=0 0 -1.5708 -> xyz=0.25 0 0 rpy=0 0 0
- joint frontRight_hip_motor_joint: origin xyz=0 0 0 rpy=0 -1.5708 -1.5708 -> xyz=0 0 0 rpy=1.5708  0 -1.5708
- joint frontRight_knee_joint: origin xyz=0.05 0 0 rpy=1.5708 0.0000 0.7854 -> xyz=0.1 0 0 rpy=1.5708 0   0
