Commit message: Update DH parameters

File: src/quadruped_arm_motion/urdf/quadruped_arm_robot_dynamics.urdf (robot description, URDF)
Before this commit: robot quadruped_arm_robot, 29 links, 28 joints
Links:
- link M0_big: mass 0.15800 -> 0.670

File: src/quadruped_arm_motion/urdf/quadruped_arm_robot_fixedbase.urdf (robot description, URDF)
Before this commit: robot quadruped_arm_robot, 23 links, 22 joints
Links:
- link M0_big: mass 0.15800 -> 0.670

Commit message: Solve issues serial communication

File: src/quadruped_arm_motion/urdf/quadruped_arm_robot_dynamics.urdf (robot description, URDF)
Before this commit: robot quadruped_arm_robot, 29 links, 28 joints
Links:
- removed link COG
- removed link Pitch_body
- removed link Roll_body
- removed link Y_body
- removed link Yaw_body
- removed link Z_body
Joints:
- removed joint Pitch_joint
- removed joint Roll_joint
- removed joint X_joint
- removed joint Y_joint
- removed joint Yaw_joint
- removed joint Z_joint
- joint articulacion1: parent Yaw_body -> base_link
- joint backLeft_hip_motor_joint: parent Yaw_body -> base_link
- joint backRight_hip_motor_joint: parent Yaw_body -> base_link
- joint endEfectorJoin: origin xyz=0.0 0 1 rpy=0 0 0 -> xyz=0.0 0 0.1 rpy=0 0 0
- joint frontLeft_hip_motor_joint: parent Yaw_body -> base_link
- joint frontRight_hip_motor_joint: parent Yaw_body -> base_link
