Commit message: Correction URDF
Is modify joints visualiation of the motor

File: src/quadruped_arm_motion/urdf/quadruped_arm_robot_Control_effort.urdf (robot description, URDF)
Before this commit: robot quadruped_arm_robot, 32 links, 31 joints
Links:
- link frontLeft_knee: mass 0.158 -> 0.001

File: src/quadruped_arm_motion/urdf/quadruped_arm_robot_control_real_effortTest_develope.urdf (robot description, URDF)
Before this commit: robot quadruped_arm_robot, 33 links, 32 joints
Links:
- added link M0_big_fixed, mass 0.158; collision mesh filename=/home/edipo/Documents/Robot_URDF3/meshes/M0.stl scale=1 1 1; visual mesh filename=/home/edipo/Documents/Robot_URDF3/meshes/M0.stl scale=1 1 1
- added link M2_100_fixed, mass 0.158; collision mesh filename=/home/edipo/Documents/Robot_URDF3/meshes/arqticulacion3.stl; visual mesh filename=/home/edipo/Documents/Robot_URDF3/meshes/arqticulacion3.stl
- added link M3_50_fixed, mass 0.158; collision mesh filename=/home/edipo/Documents/Robot_URDF3/meshes/arqticulacion4.stl; visual mesh filename=/home/edipo/Documents/Robot_URDF3/meshes/arqticulacion4.stl
- added link M4_50_fixed, mass 0.158; collision mesh filename=/home/edipo/Documents/Robot_URDF3/meshes/articulacion5.stl; visual mesh filename=/home/edipo/Documents/Robot_URDF3/meshes/articulacion5.stl
- added link backLeft_ankle_fixed, mass 0.158; collision mesh filename=/home/edipo/Documents/Robot_URDF3/meshes/servo_8y.stl scale=1 1 1; visual mesh filename=/home/edipo/Documents/Robot_URDF3/meshes/servo_8y.stl scale=1 1 1
- added link backLeft_hip_motor_fixed, mass 0.158; collision mesh filename=/home/edipo/Documents/Robot_URDF3/meshes/servo_8y.stl scale=1 1 1; visual mesh filename=/home/edipo/Documents/Robot_URDF3/meshes/servo_8y.stl scale=1 1 1
- added link backLeft_knee_fixed, mass 0.158; collision mesh filename=/home/edipo/Documents/Robot_URDF3/meshes/servo_8y.stl scale=1 1 1; visual mesh filename=/home/edipo/Documents/Robot_URDF3/meshes/servo_8y.stl scale=1 1 1
- added link backRight_ankle_fixed, mass 0.158; collision mesh filename=/home/edipo/Documents/Robot_URDF3/meshes/servo_8y.stl scale=1 1 1; visual mesh filename=/home/edipo/Documents/Robot_URDF3/meshes/servo_8y.stl scale=1 1 1
- added link backRight_hip_motor_fixed, mass 0.158; collision mesh filename=/home/edipo/Documents/Robot_URDF3/meshes/servo_7y.stl scale=1 1 1; visual mesh filename=/home/edipo/Documents/Robot_URDF3/meshes/servo_7y.stl scale=1 1 1
- added link backRight_knee_fixed, mass 0.158; collision mesh filename=/home/edipo/Documents/Robot_URDF3/meshes/servo_8y.stl scale=1 1 1; visual mesh filename=/home/edipo/Documents/Robot_URDF3/meshes/servo_8y.stl scale=1 1 1
- added link frontLeft_ankle_fixed, mass 0.158; collision mesh filename=/home/edipo/Documents/Robot_URDF3/meshes/servo_8y.stl scale=1 1 1; visual mesh filename=/home/edipo/Documents/Robot_URDF3/meshes/servo_8y.stl scale=1 1 1
- added link frontLeft_hip_motor_fixed, mass 0.158; collision mesh filename=/home/edipo/Documents/Robot_URDF3/meshes/servo_8y.stl scale=1 1 1; visual mesh filename=/home/edipo/Documents/Robot_URDF3/meshes/servo_8y.stl scale=1 1 1
- added link frontLeft_knee_fixed, mass 0.158; collision mesh filename=/home/edipo/Documents/Robot_URDF3/meshes/servo_8y.stl scale=1 1 1; visual mesh filename=/home/edipo/Documents/Robot_URDF3/meshes/servo_8y.stl scale=1 1 1
- added link frontRight_ankle_fixed, mass 0.158; collision mesh filename=/home/edipo/Documents/Robot_URDF3/meshes/servo_8y.stl scale=1 1 1; visual mesh filename=/home/edipo/Documents/Robot_URDF3/meshes/servo_8y.stl scale=1 1 1
- added link frontRight_hip_motor_fixed, mass 0.158; collision mesh filename=/home/edipo/Documents/Robot_URDF3/meshes/servo_7y.stl scale=1 1 1; visual mesh filename=/home/edipo/Documents/Robot_URDF3/meshes/servo_7y.stl scale=1 1 1
- added link frontRight_knee_fixed, mass 0.158; collision mesh filename=/home/edipo/Documents/Robot_URDF3/meshes/servo_8y.stl scale=1 1 1; visual mesh filename=/home/edipo/Documents/Robot_URDF3/meshes/servo_8y.stl scale=1 1 1
- link M0_big: mass 0.158 -> 0.05; geometry collision box size=0.125 0.04 0.02; visual box size=0.125 0.04 0.02
- link M2_100: mass 0.158 -> 0.05; geometry collision box size=0.125 0.04 0.02; visual box size=0.125 0.04 0.02
- link M3_50: mass 0.158 -> 0.05; geometry collision box size=0.125 0.04 0.02; visual box size=0.125 0.04 0.02
- link M4_50: mass 0.158 -> 0.05; geometry collision box size=0.125 0.04 0.02; visual box size=0.125 0.04 0.02
- link backLeft_ankle: mass 0.158 -> 0.05; geometry collision box size=0.125 0.04 0.02; visual box size=0.125 0.04 0.02
- link backLeft_hip_motor: mass 0.158 -> 0.05; geometry collision box size=0.125 0.04 0.02; visual box size=0.125 0.04 0.02
- link backLeft_knee: mass 0.158 -> 0.05; geometry collision box size=0.125 0.04 0.02; visual box size=0.125 0.04 0.02
- link backRight_ankle: mass 0.158 -> 0.05; geometry collision box size=0.125 0.04 0.02; visual box size=0.125 0.04 0.02
- link backRight_hip_motor: mass 0.158 -> 0.05; geometry collision box size=0.125 0.04 0.02; visual box size=0.125 0.04 0.02
- link backRight_knee: mass 0.158 -> 0.05; geometry collision box size=0.125 0.04 0.02; visual box size=0.125 0.04 0.02
- link frontLeft_ankle: mass 0.158 -> 0.05; geometry collision box size=0.125 0.04 0.02; visual box size=0.125 0.04 0.02
- link frontLeft_hip_motor: mass 0.158 -> 0.001; geometry collision cylinder length=0.05 radius=0.015; visual cylinder length=0.05 radius=0.015
- link frontLeft_knee: mass 0.158 -> 0.05; geometry collision box size=0.125 0.04 0.02; visual box size=0.125 0.04 0.02
- link frontRight_ankle: mass 0.158 -> 0.05; geometry collision box size=0.125 0.04 0.02; visual box size=0.125 0.04 0.02
- link frontRight_hip_motor: mass 0.158 -> 0.05; geometry collision box size=0.125 0.04 0.02; visual box size=0.125 0.04 0.02
- link frontRight_knee: mass 0.158 -> 0.05; geometry collision box size=0.125 0.04 0.02; visual box size=0.125 0.04 0.02
Joints:
- added joint articulacion1_fixed: type fixed, parent base_link, child M0_big_fixed, origin xyz=0 -0.03 0.1 rpy=0 0 0, axis 0 0 1, limit lower=-1.14 upper=1.14 effort=19.03325 velocity=1
- added joint articulacion3_fixed: type fixed, parent Connector_1, child M2_100_fixed, origin xyz=0.012964 -0.281387 0.005002 rpy=3.141593 3.141593 0.098574, axis 0 0 1, limit lower=-1.14 upper=1.14 effort=19.03325 velocity=1
- added joint articulacion4_fixed: type fixed, parent M2_100, child M3_50_fixed, origin xyz=0.012922 0.071422 -0.000218 rpy=-2.768763 4.595309 -0.481668, axis 0 0 1, limit lower=-1.14 upper=1.14 effort=19.03325 velocity=1
- added joint articulacion5_fixed: type fixed, parent Connector_2, child M4_50_fixed, origin xyz=-0.007231 -0.062830 0.290000 rpy=1.570798 3.141596 1.134464, axis 0 0 1, limit lower=-1.14 upper=1.14 effort=19.03325 velocity=1
- added joint backLeft_ankle_joint_fixed: type fixed, parent backLeft_connector, child backLeft_ankle_fixed, origin xyz=0.07 0 0 rpy=-0.0032  0  1.5, axis 0 0 1, limit lower=-3.14 upper=3.14 effort=50.88 velocity=1
- added joint backLeft_hip_motor_joint_fixed: type fixed, parent base_link, child backLeft_hip_motor_fixed, origin xyz=-0.19 0.03 0.03 rpy=0 1.5708 0, axis 0 0 1, limit lower=-3.14 upper=3.14 effort=50.88 velocity=1
- added joint backLeft_knee_joint_fixed: type fixed, parent backLeft_hip_motor, child backLeft_knee_fixed, origin xyz=0.030 0.055 0.01 rpy=1.5708 0 0, axis 0 0 1, limit lower=-1.57 upper=1.57 effort=50.88 velocity=1
- added joint backRight_ankle_joint_fixed: type fixed, parent backRight_connector, child backRight_ankle_fixed, origin xyz=0.07 0 0 rpy=-0.0032  0  1.5, axis 0 0 1, limit lower=-3.14 upper=3.14 effort=50.88 velocity=1
- added joint backRight_hip_motor_joint_fixed: type fixed, parent base_link, child backRight_hip_motor_fixed, origin xyz=-0.19 -0.085 0.03 rpy=0 1.5708 0, axis 0 0 1, limit lower=-3.14 upper=3.14 effort=50.88 velocity=1
- added joint backRight_knee_joint_fixed: type fixed, parent backRight_hip_motor, child backRight_knee_fixed, origin xyz=0.035 -0.045 0.01 rpy=1.5708 0 0, axis 0 0 1, limit lower=-1.57 upper=1.57 effort=50.88 velocity=1
- added joint frontLeft_ankle_joint_fixed: type fixed, parent frontLeft_connector, child frontLeft_ankle_fixed, origin xyz=0.07 0 0 rpy=-0.0032  0  1.5, axis 0 0 1, limit lower=-3.14 upper=3.14 effort=50.88 velocity=1
- added joint frontLeft_hip_motor_joint_fixed: type fixed, parent base_link, child frontLeft_hip_motor_fixed, origin xyz=0.15 0.03 0.03 rpy=0 1.5708 0, axis 0 0 1, limit lower=-3.14 upper=3.14 effort=50.88 velocity=1
- added joint frontLeft_knee_joint_fixed: type fixed, parent frontLeft_hip_motor, child frontLeft_knee_fixed, origin xyz=0.030 0.055 -0.015 rpy=1.5708 0 0, axis 0 0 1, limit lower=-1.57 upper=1.57 effort=50.88 velocity=1
- added joint frontRight_ankle_joint_fixed: type fixed, parent frontRight_connector, child frontRight_ankle_fixed, origin xyz=0.07 0 0 rpy=-0.0032  0  1.5, axis 0 0 1, limit lower=-3.14 upper=3.14 effort=50.88 velocity=1
- added joint frontRight_hip_motor_joint_fixed: type fixed, parent base_link, child frontRight_hip_motor_fixed, origin xyz=0.15 -0.085 0.03 rpy=0 1.5708 0, axis 0 0 1, limit lower=-3.14 upper=3.14 effort=50.88 velocity=1
- added joint frontRight_knee_joint_fixed: type fixed, parent frontRight_hip_motor, child frontRight_knee_fixed, origin xyz=0.035 -0.045 -0.01 rpy=1.5708 0 0, axis 0 0 1, limit lower=-1.57 upper=1.57 effort=50.88 velocity=1
- joint articulacion1: origin xyz=0 -0.03 0.1 rpy=0 0 0 -> xyz=0 0 0 rpy=0 0 0; parent base_link -> M0_big_fixed
- joint articulacion3: origin xyz=0.012964 -0.281387 0.005002 rpy=3.141593 3.141593 0.098574 -> xyz=0 0 0 rpy=0 0 0; parent Connector_1 -> M2_100_fixed
- joint articulacion4: origin xyz=0.012922 0.071422 -0.000218 rpy=-2.768763 4.595309 -0.481668 -> xyz=0 0 0 rpy=0 0 0; parent M2_100 -> M3_50_fixed
- joint articulacion5: origin xyz=-0.007231 -0.062830 0.290000 rpy=1.570798 3.141596 1.134464 -> xyz=0 0 0 rpy=0 0 0; parent Connector_2 -> M4_50_fixed
- joint backLeft_ankle_joint: origin xyz=0.07 0 0 rpy=-0.0032  0  1.5 -> xyz=0.0 0 0 rpy=0 0 0; parent backLeft_connector -> backLeft_ankle_fixed
- joint backLeft_hip_motor_joint: origin xyz=-0.19 0.03 0.03 rpy=0 1.5708 0 -> xyz=0 0 0 rpy=0 0 0; parent base_link -> backLeft_hip_motor_fixed
- joint backLeft_knee_joint: origin xyz=0.030 0.055 0.01 rpy=1.5708 0 0 -> xyz=0 0 0 rpy=0 0 0; parent backLeft_hip_motor -> backLeft_knee_fixed
- joint backRight_ankle_joint: origin xyz=0.07 0 0 rpy=-0.0032  0  1.5 -> xyz=0.0 0 0 rpy=0 0 0; parent backRight_connector -> backRight_ankle_fixed
- joint backRight_hip_motor_joint: origin xyz=-0.19 -0.085 0.03 rpy=0 1.5708 0 -> xyz=0 0 0 rpy=0 0 0; parent base_link -> backRight_hip_motor_fixed
- joint backRight_knee_joint: origin xyz=0.035 -0.045 0.01 rpy=1.5708 0 0 -> xyz=0 0 0 rpy=0 0 0; parent backRight_hip_motor -> backRight_knee_fixed
- joint frontLeft_ankle_joint: origin xyz=0.07 0 0 rpy=-0.0032  0  1.5 -> xyz=0.0 0 0 rpy=0 0 0; parent frontLeft_connector -> frontLeft_ankle_fixed
- joint frontLeft_hip_motor_joint: origin xyz=0.15 0.03 0.03 rpy=0 1.5708 0 -> xyz=0 0 0 rpy=0 0 0; parent base_link -> frontLeft_hip_motor_fixed
- joint frontLeft_knee_joint: origin xyz=0.030 0.055 -0.015 rpy=1.5708 0 0 -> xyz=0 0 0 rpy=0 0 0; parent frontLeft_hip_motor -> frontLeft_knee_fixed
- joint frontRight_ankle_joint: origin xyz=0.07 0 0 rpy=-0.0032  0  1.5 -> xyz=0 0 0 rpy=0 0 0; parent frontRight_connector -> frontRight_ankle_fixed
- joint frontRight_hip_motor_joint: origin xyz=0.15 -0.085 0.03 rpy=0 1.5708 0 -> xyz=0 0 0 rpy=0 0 0; parent base_link -> frontRight_hip_motor_fixed
- joint frontRight_knee_joint: origin xyz=0.035 -0.045 -0.01 rpy=1.5708 0 0 -> xyz=0 0 0 rpy=0 0 0; parent frontRight_hip_motor -> frontRight_knee_fixed
