Commit message: Fixed joints locations, pending to improve visual of foots

File: src/quadruped_arm_motion/urdf/quadruped_arm_robot_control_real_effort.urdf (robot description, URDF)
Before this commit: robot quadruped_arm_robot, 32 links, 31 joints
Links:
- removed link Motor_square_2
- removed link Motor_square_3
- added link M0_big_fixed, mass 0.158; collision mesh filename=/home/edipo/Documents/Robot_URDF3/meshes/M0.stl scale=1 1 1; visual mesh filename=/home/edipo/Documents/Robot_URDF3/meshes/M0.stl scale=1 1 1
- added link M2_100_fixed, mass 0.158; collision mesh filename=/home/edipo/Documents/Robot_URDF3/meshes/arqticulacion3.stl; visual mesh filename=/home/edipo/Documents/Robot_URDF3/meshes/arqticulacion3.stl
- added link M3_50_fixed, mass 0.158; collision mesh filename=/home/edipo/Documents/Robot_URDF3/meshes/arqticulacion4.stl; visual mesh filename=/home/edipo/Documents/Robot_URDF3/meshes/arqticulacion4.stl
- added link M4_50_fixed, mass 0.158; collision mesh filename=/home/edipo/Documents/Robot_URDF3/meshes/articulacion5.stl; visual mesh filename=/home/edipo/Documents/Robot_URDF3/meshes/articulacion5.stl
- added link backLeft_ankle_fixed, mass 0.158; collision mesh filename=/home/edipo/Documents/Robot_URDF3/meshes/servo_8y.stl scale=1 1 1; visual mesh filename=/home/edipo/Documents/Robot_URDF3/meshes/servo_8y.stl scale=1 1 1
- added link backLeft_hip_motor_fixed, mass 0.158; collision mesh filename=/home/edipo/Documents/Robot_URDF3/meshes/servo_8y.stl scale=1 1 1; visual mesh filename=/home/edipo/Documents/Robot_URDF3/meshes/servo_8y.stl scale=1 1 1
- added link backRight_ankle_fixed, mass 0.158; collision mesh filename=/home/edipo/Documents/Robot_URDF3/meshes/servo_8y.stl scale=1 1 1; visual mesh filename=/home/edipo/Documents/Robot_URDF3/meshes/servo_8y.stl scale=1 1 1
- added link backRight_hip_motor_fixed, mass 0.158; collision mesh filename=/home/edipo/Documents/Robot_URDF3/meshes/servo_7y.stl scale=1 1 1; visual mesh filename=/home/edipo/Documents/Robot_URDF3/meshes/servo_7y.stl scale=1 1 1
- added link camera_link, mass 0.01; collision box size=0.05 0.05 0.05; visual box size=0.04 0.04 0.04
- added link frontLeft_ankle_fixed, mass 0.158; collision mesh filename=/home/edipo/Documents/Robot_URDF3/meshes/servo_8y.stl scale=1 1 1; visual mesh filename=/home/edipo/Documents/Robot_URDF3/meshes/servo_8y.stl scale=1 1 1
- added link frontLeft_hip_motor_fixed, mass 0.158; collision mesh filename=/home/edipo/Documents/Robot_URDF3/meshes/servo_8y.stl scale=1 1 1; visual mesh filename=/home/edipo/Documents/Robot_URDF3/meshes/servo_8y.stl scale=1 1 1
- added link frontRight_ankle_fixed, mass 0.158; collision mesh filename=/home/edipo/Documents/Robot_URDF3/meshes/servo_8y.stl scale=1 1 1; visual mesh filename=/home/edipo/Documents/Robot_URDF3/meshes/servo_8y.stl scale=1 1 1
- added link frontRight_hip_motor_fixed, mass 0.158; collision mesh filename=/home/edipo/Documents/Robot_URDF3/meshes/servo_7y.stl scale=1 1 1; visual mesh filename=/home/edipo/Documents/Robot_URDF3/meshes/servo_7y.stl scale=1 1 1
- added link imu1_link, mass 0.001; collision box size=0.05 0.05 0.05; visual box size=0.005 0.005 0.005
- added link imu2_link, mass 0.001; collision box size=0.05 0.05 0.05; visual box size=0.005 0.005 0.005
- link Connector_1: geometry collision mesh filename=/home/edipo/Documents/Robot_URDF3/meshes/arqticulacion2.stl; visual mesh filename=/home/edipo/Documents/Robot_URDF3/meshes/arqticulacion2.stl
- link Connector_2: geometry collision mesh filename=/home/edipo/Documents/Robot_URDF3/meshes/connector2.stl; visual mesh filename=/home/edipo/Documents/Robot_URDF3/meshes/connector2.stl
- link M0_big: mass 0.158 -> 0.05; geometry collision box size=0.06 0.06 0.06
- link M1_100: mass 0.158 -> 0.001; geometry collision box size=0.05 0.05 0.05
- link M2_100: mass 0.08158 -> 0.05; geometry collision box size=0.06 0.06 0.06
- link M3_50: mass 0.08158 -> 0.05; geometry collision box size=0.06 0.06 0.06
- link M4_50: mass 0.08158 -> 0.05; geometry collision box size=0.06 0.06 0.06
- link Motor_square: mass 0.08158 -> 0.001; geometry visual mesh filename=/home/edipo/Documents/Robot_URDF3/meshes/Motor_square.stl
- link backLeft_ankle: mass 0.158 -> 0.05; geometry collision box size=0.06 0.06 0.06
- link backLeft_foot: geometry collision mesh filename=/home/edipo/Documents/Robot_URDF3/meshes/foot_4.stl scale=1 1 1; visual mesh filename=/home/edipo/Documents/Robot_URDF3/meshes/foot_4.stl scale=1 1 1
- link backLeft_hip_motor: mass 0.158 -> 0.05; geometry collision box size=0.06 0.06 0.06
- link backRight_ankle: mass 0.158 -> 0.05; geometry collision box size=0.06 0.06 0.06
- link backRight_foot: geometry collision mesh filename=/home/edipo/Documents/Robot_URDF3/meshes/foot_4.stl scale=1 1 1; visual mesh filename=/home/edipo/Documents/Robot_URDF3/meshes/foot_4.stl scale=1 1 1
- link backRight_hip_motor: mass 0.158 -> 0.05; geometry collision box size=0.06 0.06 0.06
- link frontLeft_ankle: mass 0.158 -> 0.05; geometry collision box size=0.05 0.05 0.05
- link frontLeft_hip_motor: mass 0.158 -> 0.001; geometry collision box size=0.06 0.06 0.06
- link frontRight_ankle: mass 0.158 -> 0.05; geometry collision box size=0.06 0.06 0.06
- link frontRight_foot: geometry collision mesh filename=/home/edipo/Documents/Robot_URDF3/meshes/foot_4.stl scale=1 1 1; visual mesh filename=/home/edipo/Documents/Robot_URDF3/meshes/foot_4.stl scale=1 1 1
- link frontRight_hip_motor: mass 0.158 -> 0.05; geometry collision box size=0.06 0.06 0.06
Joints:
- removed joint Motor_square_2_Join
- removed joint Motor_square_3_Join
- added joint articulacion1_fixed: type fixed, parent base_link, child M0_big_fixed, origin xyz=0 -0.03 0.1 rpy=0 0 0, axis 0 0 1
- added joint articulacion3_fixed: type fixed, parent Connector_1, child M2_100_fixed, origin xyz=-0.004 -0.335 0.0059 rpy=3.141593 3.141593 0.098574, axis 0 0 1
- added joint articulacion4_fixed: type fixed, parent M2_100, child M3_50_fixed, origin xyz=0.012922 0.071422 -0.000218 rpy=-2.768763 4.595309 -0.481668, axis 0 0 1
- added joint articulacion5_fixed: type fixed, parent Connector_2, child M4_50_fixed, origin xyz=-0.03 -0.062830 0.290000 rpy=1.570798 3.141596 -0.4, axis 0 0 1
- added joint backLeft_ankle_joint_fixed: type fixed, parent backLeft_connector, child backLeft_ankle_fixed, origin xyz=0.07 0 0 rpy=-0.0032  0  1.5, axis 0 0 1
- added joint backLeft_hip_motor_joint_fixed: type fixed, parent base_link, child backLeft_hip_motor_fixed, origin xyz=-0.19 0.03 0.03 rpy=0 1.5708 0, axis 0 0 1
- added joint backRight_ankle_joint_fixed: type fixed, parent backRight_connector, child backRight_ankle_fixed, origin xyz=0.07 0 0 rpy=-0.0032  0  1.5, axis 0 0 1
- added joint backRight_hip_motor_joint_fixed: type fixed, parent base_link, child backRight_hip_motor_fixed, origin xyz=-0.19 -0.085 0.03 rpy=0 1.5708 0, axis 0 0 1
- added joint camera_fixed_joint: type fixed, parent base_link, child camera_link, origin xyz=0.17 -0.03 0.05 rpy=0 0 0
- added joint frontLeft_ankle_joint_fixed: type fixed, parent frontLeft_connector, child frontLeft_ankle_fixed, origin xyz=0.07 0 0 rpy=-0.0032  0  1.5, axis 0 0 1
- added joint frontLeft_hip_motor_joint_fixed: type fixed, parent base_link, child frontLeft_hip_motor_fixed, origin xyz=0.15 0.03 0.03 rpy=0 1.5708 0, axis 0 0 1
- added joint frontRight_ankle_joint_fixed: type fixed, parent frontRight_connector, child frontRight_ankle_fixed, origin xyz=0.07 0 0 rpy=-0.0032  0  1.5, axis 0 0 1
- added joint frontRight_hip_motor_joint_fixed: type fixed, parent base_link, child frontRight_hip_motor_fixed, origin xyz=0.15 -0.085 0.03 rpy=0 1.5708 0, axis 0 0 1
- added joint imu1_fixed_joint: type fixed, parent base_link, child imu1_link, origin xyz=0.12 -0.01 0.05 rpy=0 0 0
- added joint imu2_fixed_joint: type fixed, parent base_link, child imu2_link, origin xyz=0.12 -0.05 0.05 rpy=0 0 0
- joint Connector_1_join: origin xyz=0.0 0 0 rpy=0 0 0 -> xyz=0 0 -0.000000 rpy=3.141593 3.141593 3.141593
- joint Connector_2_join: origin xyz=0.0 0 0 rpy=0 0 0 -> xyz=-0.005625 0.070702 -0.01 rpy=3.107243 3.130790 -2.619391
- joint Motor_square_Join: origin xyz=0.0 0 0.05 rpy=0 0 0 -> xyz=0.000000 0.000000 -0.050000 rpy=3.141592 3.141592 0.000000
- joint articulacion1: origin xyz=0 -0.03 0.1 rpy=0 0 0 -> xyz=0 0 0 rpy=0 3.14 0; parent base_link -> M0_big_fixed
- joint articulacion2: origin xyz=0.0 0 0.05 rpy=-1.5708 0.0 0 -> xyz=0.000000 -0.000000 -0.020000 rpy=-1.588239 3.142206 -3.106692
- joint articulacion3: origin xyz=0.0 -0.25  0   rpy=0 0 0.5 -> xyz=-0.02 -0.03 -0 rpy=0 0 0; parent Connector_1 -> M2_100_fixed
- joint articulacion4: origin xyz=0 -0.07 0 rpy= 0 1.5708 0 -> xyz=0 0 0 rpy=0 3 0; parent Motor_square_2 -> M3_50_fixed
- joint articulacion5: origin xyz=0 0 0.05 rpy=-1.5708 0 0 -> xyz=0 0 0 rpy=0 0 0; parent Motor_square_3 -> M4_50_fixed
- joint backLeft_ankle_joint: origin xyz=0.07 0 0 rpy=-0.0032  -0.003  0.712 -> xyz=0.0 0 0 rpy=0 0 0; parent backLeft_connector -> backLeft_ankle_fixed
- joint backLeft_foot_joint: origin xyz=0.09 0 0 -> xyz=0  -0.04  0
- joint backLeft_hip_motor_joint: origin xyz=-0.275 0.03 0.03 rpy=0 1.5708 0 -> xyz=0 0 0 rpy=0 0 0; parent base_link -> backLeft_hip_motor_fixed
- joint backRight_ankle_joint: origin xyz=0.07 0 0 rpy=-0.0032  -0.003  0.712 -> xyz=0.0 0 0 rpy=0 0 0; parent backRight_connector -> backRight_ankle_fixed
- joint backRight_foot_joint: origin xyz=0.09 0 0 -> xyz=0  -0.04  0
- joint backRight_hip_motor_joint: origin xyz=-0.275 -0.085 0.03 rpy=0 1.5708 0 -> xyz=0 0 0 rpy=0 0 0; parent base_link -> backRight_hip_motor_fixed
- joint endEfectorJoin: origin xyz=0 0 0.1 rpy=0 0 0 -> xyz=0 -0.05 0.03 rpy=0 0 0; parent Motor_square_3 -> M4_50
- joint frontLeft_ankle_joint: origin xyz=0.07 0 0 rpy=-0.0032  -0.003  0.712 -> xyz=0.0 0 0 rpy=0 0 0; parent frontLeft_connector -> frontLeft_ankle_fixed
- joint frontLeft_foot_joint: origin xyz=0.09 0 0 rpy=0 0  -0.5 -> xyz=0  -0.04  0
- joint frontLeft_hip_motor_joint: origin xyz=0.235 0.03 0.03 rpy=0 1.5708 0 -> xyz=0 0 0 rpy=0 0 0; parent base_link -> frontLeft_hip_motor_fixed
- joint frontRight_ankle_joint: origin xyz=0.07 0 0 rpy=-0.0032  -0.003  0.712 -> xyz=0 0 0 rpy=0 0 0; parent frontRight_connector -> frontRight_ankle_fixed
- joint frontRight_foot_joint: origin xyz=0.09 0 0 -> xyz=0  -0.04  0
- joint frontRight_hip_motor_joint: origin xyz=0.235 -0.085 0.03 rpy=0 1.5708 0 -> xyz=0 0 0 rpy=0 0 0; parent base_link -> frontRight_hip_motor_fixed

File: src/quadruped_arm_motion/urdf/quadruped_arm_robot_control_real_effortTest_develope.urdf (robot description, URDF)
Before this commit: robot quadruped_arm_robot, 45 links, 44 joints
Links:
- removed link backLeft_hip_motor_fixed
- removed link backRight_hip_motor_fixed
- removed link frontLeft_hip_motor_fixed
- removed link frontRight_hip_motor_fixed
- link M0_big: geometry collision box size=0.06 0.06 0.06; visual box size=0.06 0.06 0.06
- link M1_100: geometry visual mesh filename=/home/edipo/Documents/Robot_URDF3/meshes/Motor_square.stl
- link M2_100: geometry collision box size=0.06 0.06 0.06; visual box size=0.06 0.06 0.06
- link M3_50: geometry collision box size=0.06 0.06 0.06; visual box size=0.06 0.06 0.06
- link M4_50: geometry collision box size=0.06 0.06 0.06; visual box size=0.06 0.06 0.06
- link backLeft_ankle: geometry collision sphere radius=0.015; visual sphere radius=0.015
- link backLeft_ankle_fixed: geometry collision mesh filename=/home/edipo/Documents/Robot_URDF3/meshes/servo_8y.stl scale=0.1 0.1; visual mesh filename=/home/edipo/Documents/Robot_URDF3/meshes/servo_8y.stl scale=1 1 1
- link backLeft_hip_motor: mass 0.05 -> 0.158; geometry collision mesh filename=/home/edipo/Documents/Robot_URDF3/meshes/servo_8y.stl scale=1 1 1; visual mesh filename=/home/edipo/Documents/Robot_URDF3/meshes/servo_8y.stl scale=1 1 1
- link backRight_ankle: geometry collision sphere radius=0.015; visual sphere radius=0.015
- link backRight_ankle_fixed: geometry collision mesh filename=/home/edipo/Documents/Robot_URDF3/meshes/servo_8y.stl scale=0.1 0.1; visual mesh filename=/home/edipo/Documents/Robot_URDF3/meshes/servo_8y.stl scale=1 1 1
- link backRight_hip_motor: mass 0.05 -> 0.158; geometry collision mesh filename=/home/edipo/Documents/Robot_URDF3/meshes/servo_7y.stl scale=1 1 1; visual mesh filename=/home/edipo/Documents/Robot_URDF3/meshes/servo_7y.stl scale=1 1 1
- link frontLeft_ankle: geometry collision sphere radius=0.015; visual sphere radius=0.015
- link frontLeft_ankle_fixed: geometry collision mesh filename=/home/edipo/Documents/Robot_URDF3/meshes/servo_8y.stl scale=0.1 0.1; visual mesh filename=/home/edipo/Documents/Robot_URDF3/meshes/servo_8y.stl scale=1 1 1
- link frontLeft_hip_motor: mass 0.001 -> 0.158; geometry collision mesh filename=/home/edipo/Documents/Robot_URDF3/meshes/servo_8y.stl scale=1 1 1; visual mesh filename=/home/edipo/Documents/Robot_URDF3/meshes/servo_8y.stl scale=1 1 1
- link frontRight_ankle: geometry collision sphere radius=0.015; visual sphere radius=0.015
- link frontRight_ankle_fixed: geometry collision mesh filename=/home/edipo/Documents/Robot_URDF3/meshes/servo_8y.stl scale=0.1 0.1; visual mesh filename=/home/edipo/Documents/Robot_URDF3/meshes/servo_8y.stl scale=1 1 1
- link frontRight_hip_motor: mass 0.05 -> 0.158; geometry collision mesh filename=/home/edipo/Documents/Robot_URDF3/meshes/servo_7y.stl scale=1 1 1; visual mesh filename=/home/edipo/Documents/Robot_URDF3/meshes/servo_7y.stl scale=1 1 1
Joints:
- removed joint backLeft_hip_motor_joint_fixed
- removed joint backRight_hip_motor_joint_fixed
- removed joint frontLeft_hip_motor_joint_fixed
- removed joint frontRight_hip_motor_joint_fixed
- joint Connector_1_join: origin xyz=-0.015 -0.025 -0.000000 rpy=3.141593 3.141593 3.141593 -> xyz=0 0 -0.000000 rpy=3.141593 3.141593 3.141593
- joint Motor_square_Join: origin xyz=0.000000 0.000000 0.050000 rpy=3.141592 3.141592 0.000000 -> xyz=0.000000 0.000000 -0.050000 rpy=3.141592 3.141592 0.000000
- joint articulacion1: limit lower=-1.14 upper=1.14 effort=19.03325 velocity=1 -> lower=-1.14 upper=1.14 effort=5000 velocity=1; origin xyz=0 0 0 rpy=0 0 0 -> xyz=0 0 0 rpy=0 3.14 0
- joint articulacion1_fixed: limit lower=-1.14 upper=1.14 effort=19.03325 velocity=1 -> (none)
- joint articulacion2: limit lower=-1.14 upper=1.14 effort=19.03325 velocity=1 -> lower=-1.14 upper=1.14 effort=5000 velocity=1; origin xyz=0.000000 -0.000000 0.025000 rpy=1.588239 3.142206 -3.106692 -> xyz=0.000000 -0.000000 -0.020000 rpy=-1.588239 3.142206 -3.106692
- joint articulacion3: limit lower=-1.14 upper=1.14 effort=19.03325 velocity=1 -> lower=-1.14 upper=1.14 effort=5000 velocity=1; origin xyz=0 0 0 rpy=0 0 0 -> xyz=-0.02 -0.03 -0 rpy=0 0 0
- joint articulacion3_fixed: limit lower=-1.14 upper=1.14 effort=19.03325 velocity=1 -> (none); origin xyz=0.012964 -0.281387 0.005002 rpy=3.141593 3.141593 0.098574 -> xyz=-0.004 -0.335 0.0059 rpy=3.141593 3.141593 0.098574
- joint articulacion4: limit lower=-1.14 upper=1.14 effort=19.03325 velocity=1 -> lower=-1.14 upper=1.14 effort=5000 velocity=1; origin xyz=0 0 0 rpy=0 0 0 -> xyz=0 0 0 rpy=0 3 0
- joint articulacion4_fixed: limit lower=-1.14 upper=1.14 effort=19.03325 velocity=1 -> (none)
- joint articulacion5: limit lower=-1.14 upper=1.14 effort=19.03325 velocity=1 -> lower=-1.14 upper=1.14 effort=5000 velocity=1
- joint articulacion5_fixed: limit lower=-1.14 upper=1.14 effort=19.03325 velocity=1 -> (none); origin xyz=-0.007231 -0.062830 0.290000 rpy=1.570798 3.141596 -0.4 -> xyz=-0.03 -0.062830 0.290000 rpy=1.570798 3.141596 -0.4
- joint backLeft_ankle_joint: limit lower=-3.14 upper=3.14 effort=50.88 velocity=1 -> lower=-3.14 upper=3.14 effort=5000 velocity=1; origin xyz=0.0 0 0 rpy=0 0 0 -> xyz=0.07 0 0 rpy=-0.0032 0 1.5; parent backLeft_ankle_fixed -> backLeft_connector
- joint backLeft_ankle_joint_fixed: limit lower=-3.14 upper=3.14 effort=50.88 velocity=1 -> lower=-3.14 upper=3.14 effort=5000 velocity=1; type fixed -> revolute
- joint backLeft_hip_motor_joint: limit lower=-3.14 upper=3.14 effort=50.88 velocity=1 -> lower=-3.14 upper=3.14 effort=5000 velocity=1; origin xyz=0 0 0 rpy=0 0 0 -> xyz=-0.19 0.03 0.03 rpy=0 1.5708 0; parent backLeft_hip_motor_fixed -> base_link
- joint backLeft_knee_joint: limit lower=-1.57 upper=1.57 effort=50.88 velocity=1 -> lower=-1.57 upper=1.57 effort=5000 velocity=1
- joint backRight_ankle_joint: limit lower=-3.14 upper=3.14 effort=50.88 velocity=1 -> lower=-3.14 upper=3.14 effort=5000 velocity=1; origin xyz=0.0 0 0 rpy=0 0 0 -> xyz=0.07 0 0 rpy=-0.0032 0 1.5; parent backRight_ankle_fixed -> backRight_connector
- joint backRight_ankle_joint_fixed: limit lower=-3.14 upper=3.14 effort=50.88 velocity=1 -> lower=-3.14 upper=3.14 effort=5000 velocity=1; type fixed -> revolute
- joint backRight_hip_motor_joint: limit lower=-3.14 upper=3.14 effort=50.88 velocity=1 -> lower=-3.14 upper=3.14 effort=5000 velocity=1; origin xyz=0 0 0 rpy=0 0 0 -> xyz=-0.19 -0.085 0.03 rpy=0 1.5708 0; parent backRight_hip_motor_fixed -> base_link
- joint backRight_knee_joint: limit lower=-1.57 upper=1.57 effort=50.88 velocity=1 -> lower=-1.57 upper=1.57 effort=5000 velocity=1
- joint frontLeft_ankle_joint: limit lower=-3.14 upper=3.14 effort=50.88 velocity=1 -> lower=-3.14 upper=3.14 effort=5000 velocity=1; origin xyz=0.0 0 0 rpy=0 0 0 -> xyz=0.07 0 0 rpy=-0.0032 0 1.5; parent frontLeft_ankle_fixed -> frontLeft_connector
- joint frontLeft_ankle_joint_fixed: limit lower=-3.14 upper=3.14 effort=50.88 velocity=1 -> lower=-3.14 upper=3.14 effort=5000 velocity=1; type fixed -> revolute
- joint frontLeft_hip_motor_joint: limit lower=-3.14 upper=3.14 effort=50.88 velocity=1 -> lower=-3.14 upper=3.14 effort=5000 velocity=1; origin xyz=0 0 0 rpy=0 0 0 -> xyz=0.15 0.03 0.03 rpy=0 1.5708 0; parent frontLeft_hip_motor_fixed -> base_link
- joint frontLeft_knee_joint: limit lower=-1.57 upper=1.57 effort=50.88 velocity=1 -> lower=-1.57 upper=1.57 effort=5000 velocity=1
- joint frontRight_ankle_joint: limit lower=-3.14 upper=3.14 effort=50.88 velocity=1 -> lower=-3.14 upper=3.14 effort=5000 velocity=1; origin xyz=0 0 0 rpy=0 0 0 -> xyz=0.07 0 0 rpy=-0.0032 0 1.5; parent frontRight_ankle_fixed -> frontRight_connector
- joint frontRight_ankle_joint_fixed: limit lower=-3.14 upper=3.14 effort=50.88 velocity=1 -> lower=-3.14 upper=3.14 effort=5000 velocity=1; type fixed -> revolute
- joint frontRight_hip_motor_joint: limit lower=-3.14 upper=3.14 effort=50.88 velocity=1 -> lower=-3.14 upper=3.14 effort=5000 velocity=1; origin xyz=0 0 0 rpy=0 0 0 -> xyz=0.15 -0.085 0.03 rpy=0 1.5708 0; parent frontRight_hip_motor_fixed -> base_link
- joint frontRight_knee_joint: limit lower=-1.57 upper=1.57 effort=50.88 velocity=1 -> lower=-1.57 upper=1.57 effort=5000 velocity=1
