Commit message: Quito referencias erróneas a repos embebidos

File: src/quadruped_arm_motion/urdf/quadruped_arm_robot_control_real_effort.urdf (robot description, URDF)
Before this commit: robot quadruped_arm_robot, 45 links, 44 joints
Links:
- removed link backLeft_hip_motor_fixed
- removed link backRight_hip_motor_fixed
- removed link frontLeft_hip_motor_fixed
- removed link frontRight_hip_motor_fixed
- link M0_big: geometry collision box size=0.03 0.03 0.03; visual box size=0.03 0.03 0.03
- link M1_100: geometry visual mesh filename=/home/edipo/Documents/Robot_URDF3/meshes/Motor_square.stl
- link M2_100: geometry collision box size=0.03 0.03 0.03; visual box size=0.03 0.03 0.03
- link M3_50: geometry collision box size=0.03 0.03 0.03; visual box size=0.03 0.03 0.03
- link M4_50: geometry collision box size=0.03 0.03 0.03; visual box size=0.03 0.03 0.03
- link backLeft_ankle: geometry collision sphere radius=0.015; visual sphere radius=0.015
- link backLeft_ankle_fixed: geometry collision mesh filename=/home/edipo/Documents/Robot_URDF3/meshes/servo_8y.stl scale=0.1 0.1 0.1; visual mesh filename=/home/edipo/Documents/Robot_URDF3/meshes/servo_8y.stl scale=1 1 1
- link backLeft_connector: geometry collision box size=0.03 0.03 0.03; visual box size=0.03 0.03 0.03
- link backLeft_hip_motor: mass 0.05 -> 0.158; geometry collision mesh filename=/home/edipo/Documents/Robot_URDF3/meshes/servo_8y.stl scale=1 1 1; visual mesh filename=/home/edipo/Documents/Robot_URDF3/meshes/servo_8y.stl scale=1 1 1
- link backRight_ankle: geometry collision sphere radius=0.015; visual sphere radius=0.015
- link backRight_ankle_fixed: geometry collision mesh filename=/home/edipo/Documents/Robot_URDF3/meshes/servo_8y.stl scale=0.1 0.1 0.1; visual mesh filename=/home/edipo/Documents/Robot_URDF3/meshes/servo_8y.stl scale=1 1 1
- link backRight_connector: geometry collision box size=0.03 0.03 0.03; visual box size=0.03 0.03 0.03
- link backRight_hip_motor: mass 0.05 -> 0.158; geometry collision mesh filename=/home/edipo/Documents/Robot_URDF3/meshes/servo_7y.stl scale=1 1 1; visual mesh filename=/home/edipo/Documents/Robot_URDF3/meshes/servo_7y.stl scale=1 1 1
- link camera_link: geometry visual box size=0.04 0.04 0.04
- link frontLeft_ankle: geometry collision sphere radius=0.015; visual sphere radius=0.015
- link frontLeft_connector: geometry collision box size=0.03 0.03 0.03; visual box size=0.03 0.03 0.03
- link frontLeft_hip_motor: mass 0.001 -> 0.158; geometry collision mesh filename=/home/edipo/Documents/Robot_URDF3/meshes/servo_8y.stl scale=1 1 1; visual mesh filename=/home/edipo/Documents/Robot_URDF3/meshes/servo_8y.stl scale=1 1 1
- link frontRight_ankle: geometry collision sphere radius=0.015; visual sphere radius=0.015
- link frontRight_ankle_fixed: geometry collision mesh filename=/home/edipo/Documents/Robot_URDF3/meshes/servo_8y.stl scale=0.1 0.1 0.1; visual mesh filename=/home/edipo/Documents/Robot_URDF3/meshes/servo_8y.stl scale=1 1 1
- link frontRight_connector: geometry collision box size=0.03 0.03 0.03; visual box size=0.03 0.03 0.03
- link frontRight_hip_motor: mass 0.05 -> 0.158; geometry collision mesh filename=/home/edipo/Documents/Robot_URDF3/meshes/servo_7y.stl scale=1 1 1; visual mesh filename=/home/edipo/Documents/Robot_URDF3/meshes/servo_7y.stl scale=1 1 1
- link imu1_link: geometry visual box size=0.005 0.005 0.005
- link imu2_link: geometry visual box size=0.005 0.005 0.005
Joints:
- removed joint backLeft_hip_motor_joint_fixed
- removed joint backRight_hip_motor_joint_fixed
- removed joint frontLeft_hip_motor_joint_fixed
- removed joint frontRight_hip_motor_joint_fixed
- joint Motor_square_Join: axis 0 0 0 -> 0 0 1
- joint articulacion1: limit lower=-1.14 upper=1.14 effort=19.03325 velocity=1 -> lower=-1.14 upper=1.14 effort=49 velocity=1
- joint articulacion2: limit lower=-1.14 upper=1.14 effort=19.03325 velocity=1 -> lower=-1.14 upper=1.14 effort=15 velocity=1
- joint articulacion3: limit lower=-1.14 upper=1.14 effort=19.03325 velocity=1 -> lower=-1.14 upper=1.14 effort=15 velocity=1
- joint articulacion3_fixed: limit (none) -> lower=-1.14 upper=1.14 effort=6 velocity=1
- joint articulacion4: limit lower=-1.14 upper=1.14 effort=19.03325 velocity=1 -> lower=-1.14 upper=1.14 effort=6 velocity=1
- joint articulacion4_fixed: limit (none) -> lower=-1.14 upper=1.14 effort=6 velocity=1
- joint articulacion5: limit lower=-1.14 upper=1.14 effort=19.03325 velocity=1 -> lower=-1.14 upper=1.14 effort=6 velocity=1
- joint articulacion5_fixed: limit (none) -> lower=-1.14 upper=1.14 effort=6 velocity=1
- joint backLeft_ankle_joint: limit lower=-3.14 upper=3.14 effort=50.88 velocity=1 -> lower=-3.14 upper=3.14 effort=15 velocity=1; origin xyz=0.0 0 0 rpy=0 0 0 -> xyz=0.07 0 0 rpy=-0.0032 0 3; parent backLeft_ankle_fixed -> backLeft_connector
- joint backLeft_connectorJoin: origin xyz=0.08 0 0 rpy=0 0 0 -> xyz=0.05 0 0 rpy=0 0 0
- joint backLeft_foot_joint: origin xyz=0  -0.04  0 -> xyz=-0.04  0 0
- joint backLeft_hip_motor_joint: limit lower=-3.14 upper=3.14 effort=50.88 velocity=1 -> lower=-3.14 upper=3.14 effort=6 velocity=1; origin xyz=0 0 0 rpy=0 0 0 -> xyz=-0.19 0.03 0.03 rpy=0 1.5708 0; parent backLeft_hip_motor_fixed -> base_link
- joint backLeft_knee_joint: limit lower=-1.57 upper=1.57 effort=50.88 velocity=1 -> lower=-1.57 upper=1.57 effort=6 velocity=1
- joint backRight_ankle_joint: limit lower=-3.14 upper=3.14 effort=50.88 velocity=1 -> lower=-3.14 upper=3.14 effort=15 velocity=1; origin xyz=0.0 0 0 rpy=0 0 0 -> xyz=0.07 0 0 rpy=-0.0032 0 3; parent backRight_ankle_fixed -> backRight_connector
- joint backRight_connectorJoin: origin xyz=0.08 0 0 rpy=0 0 0 -> xyz=0.05 0 0 rpy=0 0 0
- joint backRight_foot_joint: origin xyz=0  -0.04  0 -> xyz=-0.04  0 0
- joint backRight_hip_motor_joint: limit lower=-3.14 upper=3.14 effort=50.88 velocity=1 -> lower=-3.14 upper=3.14 effort=6 velocity=1; origin xyz=0 0 0 rpy=0 0 0 -> xyz=-0.19 -0.085 0.03 rpy=0 1.5708 0; parent backRight_hip_motor_fixed -> base_link
- joint backRight_knee_joint: limit lower=-1.57 upper=1.57 effort=50.88 velocity=1 -> lower=-1.57 upper=1.57 effort=6 velocity=1
- joint frontLeft_ankle_joint: limit lower=-3.14 upper=3.14 effort=50.88 velocity=1 -> lower=-3.14 upper=3.14 effort=15 velocity=1; origin xyz=0.0 0 0 rpy=0 0 0 -> xyz=0.07 0 0 rpy=-0.0032 0 3; parent frontLeft_ankle_fixed -> frontLeft_connector
- joint frontLeft_ankle_joint_fixed: axis 0 0 1 -> (none)
- joint frontLeft_connectorJoin: origin xyz=0.08 0 0 rpy=0 0 0 -> xyz=0.05 0 0 rpy=0 0 0
- joint frontLeft_foot_joint: origin xyz=0  -0.04  0 -> xyz=-0.04  0 0
- joint frontLeft_hip_motor_joint: limit lower=-3.14 upper=3.14 effort=50.88 velocity=1 -> lower=-3.14 upper=3.14 effort=6 velocity=1; origin xyz=0 0 0 rpy=0 0 0 -> xyz=0.15 0.03 0.03 rpy=0 1.5708 0; parent frontLeft_hip_motor_fixed -> base_link
- joint frontLeft_knee_joint: limit lower=-1.57 upper=1.57 effort=50.88 velocity=1 -> lower=-1.57 upper=1.57 effort=6 velocity=1
- joint frontRight_ankle_joint: limit lower=-3.14 upper=3.14 effort=50.88 velocity=1 -> lower=-3.14 upper=3.14 effort=15 velocity=1; origin xyz=0 0 0 rpy=0 0 0 -> xyz=0.07 0 0 rpy=-0.0032 0 3; parent frontRight_ankle_fixed -> frontRight_connector
- joint frontRight_connectorJoin: origin xyz=0.08 0 0 rpy=0 0 0 -> xyz=0.05 0 0 rpy=0 0 0
- joint frontRight_foot_joint: origin xyz=0  -0.04  0 -> xyz=-0.04  0 0
- joint frontRight_hip_motor_joint: limit lower=-3.14 upper=3.14 effort=50.88 velocity=1 -> lower=-3.14 upper=3.14 effort=6 velocity=1; origin xyz=0 0 0 rpy=0 0 0 -> xyz=0.15 -0.085 0.03 rpy=0 1.5708 0; parent frontRight_hip_motor_fixed -> base_link
- joint frontRight_knee_joint: limit lower=-1.57 upper=1.57 effort=50.88 velocity=1 -> lower=-1.57 upper=1.57 effort=6 velocity=1

File: src/quadruped_arm_motion/urdf/quadruped_arm_robot_control_real_effortTest_develope.urdf (robot description, URDF)
Before this commit: robot quadruped_arm_robot, 41 links, 40 joints
Links:
- link Connector_1: geometry visual mesh filename=/home/edipo/Documents/Robot_URDF3/meshes/arqticulacion2.stl
- link M0_big: geometry collision box size=0.03 0.03 0.03; visual box size=0.03 0.03 0.03
- link M1_100: mass 0.001 -> 0.05
- link M2_100: geometry collision box size=0.03 0.03 0.03; visual box size=0.03 0.03 0.03
- link M2_100_fixed: geometry visual mesh filename=/home/edipo/Documents/Robot_URDF3/meshes/arqticulacion3.stl
- link M3_50: geometry collision box size=0.03 0.03 0.03; visual box size=0.03 0.03 0.03
- link M3_50_fixed: geometry visual mesh filename=/home/edipo/Documents/Robot_URDF3/meshes/arqticulacion4.stl
- link M4_50: geometry collision box size=0.03 0.03 0.03; visual box size=0.03 0.03 0.03
- link M4_50_fixed: geometry visual mesh filename=/home/edipo/Documents/Robot_URDF3/meshes/articulacion5.stl
- link Motor_square: mass 0.001 -> 0.05
- link backLeft_ankle_fixed: geometry visual mesh filename=/home/edipo/Documents/Robot_URDF3/meshes/servo_8y.stl scale=1 1 1
- link backLeft_connector: geometry visual box size=0.03 0.03 0.03
- link backLeft_foot: mass 0.03 -> 0.05
- link backRight_ankle_fixed: geometry collision mesh filename=/home/edipo/Documents/Robot_URDF3/meshes/servo_8y.stl scale=0.1 0.1 0.1; visual mesh filename=/home/edipo/Documents/Robot_URDF3/meshes/servo_8y.stl scale=1 1 1
- link backRight_connector: geometry collision box size=0.03 0.03 0.03; visual box size=0.03 0.03 0.03
- link backRight_foot: mass 0.03 -> 0.05
- link base_link: geometry visual mesh filename=/home/edipo/Documents/Robot_URDF3/meshes/Body.stl scale=1 1 1
- link endEfector: geometry visual box size=0.05 0.05 0.05
- link frontLeft_ankle_fixed: geometry visual mesh filename=/home/edipo/Documents/Robot_URDF3/meshes/servo_8y.stl scale=1 1 1
- link frontLeft_connector: geometry collision box size=0.03 0.03 0.03; visual box size=0.03 0.03 0.03
- link frontLeft_foot: mass 0.03 -> 0.05; geometry visual mesh filename=/home/edipo/Documents/Robot_URDF3/meshes/foot_3.stl scale=1 1 1
- link frontRight_ankle_fixed: geometry visual mesh filename=/home/edipo/Documents/Robot_URDF3/meshes/servo_8y.stl scale=1 1 1
- link frontRight_connector: geometry visual box size=0.03 0.03 0.03
- link frontRight_foot: mass 0.03 -> 0.05
- link imu1_link: mass 0.001 -> 0.05
- link imu2_link: mass 0.001 -> 0.05
Joints:
- joint Motor_square_Join: axis 0 0 0 -> 0 0 1; origin xyz=0.000000 0.000000 -0.050000 rpy=3.141592 3.141592 0.000000 -> xyz=0.000000 0.000000 -0.01000 rpy=3.141592 3.141592 0.000000
- joint articulacion1: limit lower=-1.14 upper=1.14 effort=5000 velocity=1 -> lower=-1.14 upper=1.14 effort=49 velocity=1
- joint articulacion2: limit lower=-1.14 upper=1.14 effort=5000 velocity=1 -> lower=-1.14 upper=1.14 effort=15 velocity=1; origin xyz=0.000000 -0.000000 -0.020000 rpy=-1.588239 3.142206 -3.106692 -> xyz=0.000000 -0.000000 -0.02000 rpy=-1.588239 3.142206 -3.106692
- joint articulacion3: limit lower=-1.14 upper=1.14 effort=5000 velocity=1 -> lower=-1.14 upper=1.14 effort=15 velocity=1
- joint articulacion3_fixed: limit (none) -> lower=-1.14 upper=1.14 effort=6 velocity=1
- joint articulacion4: limit lower=-1.14 upper=1.14 effort=5000 velocity=1 -> lower=-1.14 upper=1.14 effort=6 velocity=1
- joint articulacion4_fixed: limit (none) -> lower=-1.14 upper=1.14 effort=6 velocity=1
- joint articulacion5: limit lower=-1.14 upper=1.14 effort=5000 velocity=1 -> lower=-1.14 upper=1.14 effort=6 velocity=1
- joint articulacion5_fixed: limit (none) -> lower=-1.14 upper=1.14 effort=6 velocity=1
- joint backLeft_ankle_joint: limit lower=-3.14 upper=3.14 effort=5000 velocity=1 -> lower=-3.14 upper=3.14 effort=15 velocity=1; origin xyz=0.07 0 0 rpy=-0.0032 0 1.5 -> xyz=0.07 0 0 rpy=-0.0032 0 3
- joint backLeft_ankle_joint_fixed: limit lower=-3.14 upper=3.14 effort=5000 velocity=1 -> (none); type revolute -> fixed
- joint backLeft_connectorJoin: origin xyz=0.08 0 0 rpy=0 0 0 -> xyz=0.05 0 0 rpy=0 0 0
- joint backLeft_foot_joint: origin xyz=0  -0.04  0 -> xyz=-0.04  0 0
- joint backLeft_hip_motor_joint: limit lower=-3.14 upper=3.14 effort=5000 velocity=1 -> lower=-3.14 upper=3.14 effort=6 velocity=1
- joint backLeft_knee_joint: limit lower=-1.57 upper=1.57 effort=5000 velocity=1 -> lower=-1.57 upper=1.57 effort=6 velocity=1
- joint backRight_ankle_joint: limit lower=-3.14 upper=3.14 effort=5000 velocity=1 -> lower=-3.14 upper=3.14 effort=15 velocity=1; origin xyz=0.07 0 0 rpy=-0.0032 0 1.5 -> xyz=0.07 0 0 rpy=-0.0032 0 3
- joint backRight_ankle_joint_fixed: limit lower=-3.14 upper=3.14 effort=5000 velocity=1 -> (none); type revolute -> fixed
- joint backRight_connectorJoin: origin xyz=0.08 0 0 rpy=0 0 0 -> xyz=0.05 0 0 rpy=0 0 0
- joint backRight_foot_joint: origin xyz=0  -0.04  0 -> xyz=-0.04  0 0
- joint backRight_hip_motor_joint: limit lower=-3.14 upper=3.14 effort=5000 velocity=1 -> lower=-3.14 upper=3.14 effort=6 velocity=1
- joint backRight_knee_joint: limit lower=-1.57 upper=1.57 effort=5000 velocity=1 -> lower=-1.57 upper=1.57 effort=6 velocity=1
- joint camera_fixed_joint: origin xyz=0.17 -0.03 0.05 rpy=0 0 0 -> xyz=0.17 -0.03 0.05 rpy=0 1.578 0
- joint frontLeft_ankle_joint: limit lower=-3.14 upper=3.14 effort=5000 velocity=1 -> lower=-3.14 upper=3.14 effort=15 velocity=1; origin xyz=0.07 0 0 rpy=-0.0032 0 1.5 -> xyz=0.07 0 0 rpy=-0.0032 0 3
- joint frontLeft_ankle_joint_fixed: axis 0 0 1 -> (none); limit lower=-3.14 upper=3.14 effort=5000 velocity=1 -> (none); type revolute -> fixed
- joint frontLeft_connectorJoin: origin xyz=0.08 0 0 rpy=0 0 0 -> xyz=0.05 0 0 rpy=0 0 0
- joint frontLeft_foot_joint: origin xyz=0  -0.04  0 -> xyz=-0.04  0 0
- joint frontLeft_hip_motor_joint: limit lower=-3.14 upper=3.14 effort=5000 velocity=1 -> lower=-3.14 upper=3.14 effort=6 velocity=1
- joint frontLeft_knee_joint: limit lower=-1.57 upper=1.57 effort=5000 velocity=1 -> lower=-1.57 upper=1.57 effort=6 velocity=1
- joint frontRight_ankle_joint: limit lower=-3.14 upper=3.14 effort=5000 velocity=1 -> lower=-3.14 upper=3.14 effort=15 velocity=1; origin xyz=0.07 0 0 rpy=-0.0032 0 1.5 -> xyz=0.07 0 0 rpy=-0.0032 0 3
- joint frontRight_ankle_joint_fixed: limit lower=-3.14 upper=3.14 effort=5000 velocity=1 -> (none); type revolute -> fixed
- joint frontRight_connectorJoin: origin xyz=0.08 0 0 rpy=0 0 0 -> xyz=0.05 0 0 rpy=0 0 0
- joint frontRight_foot_joint: origin xyz=0  -0.04  0 -> xyz=-0.04  0 0
- joint frontRight_hip_motor_joint: limit lower=-3.14 upper=3.14 effort=5000 velocity=1 -> lower=-3.14 upper=3.14 effort=6 velocity=1
- joint frontRight_knee_joint: limit lower=-1.57 upper=1.57 effort=5000 velocity=1 -> lower=-1.57 upper=1.57 effort=6 velocity=1
