Commit message: Delete no neccesarry vizualisation

File: src/quadruped_arm_motion/urdf/quadruped_arm_robot_control_real_effortTest_develope.urdf (robot description, URDF)
Before this commit: robot quadruped_arm_robot, 49 links, 48 joints
Links:
- removed link backLeft_knee_fixed
- removed link backRight_knee_fixed
- removed link frontLeft_knee_fixed
- removed link frontRight_knee_fixed
- link M0_big: geometry 
- link M2_100: geometry 
- link M3_50: geometry 
- link M4_50: geometry 
- link backLeft_ankle: geometry 
- link backLeft_hip_motor: geometry 
- link backLeft_knee: mass 0.05 -> 0.158; geometry collision mesh filename=/home/edipo/Documents/Robot_URDF3/meshes/servo_8y.stl scale=1 1 1; visual mesh filename=/home/edipo/Documents/Robot_URDF3/meshes/servo_8y.stl scale=1 1 1
- link backRight_ankle: geometry 
- link backRight_hip_motor: geometry 
- link backRight_knee: mass 0.05 -> 0.158; geometry collision mesh filename=/home/edipo/Documents/Robot_URDF3/meshes/servo_8y.stl scale=1 1 1; visual mesh filename=/home/edipo/Documents/Robot_URDF3/meshes/servo_8y.stl scale=1 1 1
- link frontLeft_ankle: geometry 
- link frontLeft_hip_motor: geometry 
- link frontLeft_knee: mass 0.05 -> 0.158; geometry collision mesh filename=/home/edipo/Documents/Robot_URDF3/meshes/servo_8y.stl scale=1 1 1; visual mesh filename=/home/edipo/Documents/Robot_URDF3/meshes/servo_8y.stl scale=1 1 1
- link frontRight_ankle: geometry 
- link frontRight_hip_motor: geometry 
- link frontRight_knee: mass 0.05 -> 0.158; geometry collision mesh filename=/home/edipo/Documents/Robot_URDF3/meshes/servo_8y.stl scale=1 1 1; visual mesh filename=/home/edipo/Documents/Robot_URDF3/meshes/servo_8y.stl scale=1 1 1
Joints:
- removed joint backLeft_knee_joint_fixed
- removed joint backRight_knee_joint_fixed
- removed joint frontLeft_knee_joint_fixed
- removed joint frontRight_knee_joint_fixed
- joint articulacion5_fixed: origin xyz=-0.007231 -0.062830 0.290000 rpy=1.570798 3.141596 1.134464 -> xyz=-0.007231 -0.062830 0.290000 rpy=1.570798 3.141596 -0.4
- joint backLeft_knee_joint: origin xyz=0 0 0 rpy=0 0 0 -> xyz=0.030 0.055 0.01 rpy=1.5708 0 0; parent backLeft_knee_fixed -> backLeft_hip_motor
- joint backRight_knee_joint: origin xyz=0 0 0 rpy=0 0 0 -> xyz=0.035 -0.045 0.01 rpy=1.5708 0 0; parent backRight_knee_fixed -> backRight_hip_motor
- joint endEfectorJoin: origin xyz=0 -0.05 -0.03 rpy=0 0 0 -> xyz=0 -0.05 0.03 rpy=0 0 0
- joint frontLeft_knee_joint: origin xyz=0 0 0 rpy=0 0 0 -> xyz=0.030 0.055 -0.015 rpy=1.5708 0 0; parent frontLeft_knee_fixed -> frontLeft_hip_motor
- joint frontRight_knee_joint: origin xyz=0 0 0 rpy=0 0 0 -> xyz=0.035 -0.045 -0.01 rpy=1.5708 0 0; parent frontRight_knee_fixed -> frontRight_hip_motor

Commit message: Fix camara location

File: src/quadruped_arm_motion/urdf/quadruped_arm_robot_control_real_effortTest_develope.urdf (robot description, URDF)
Before this commit: robot quadruped_arm_robot, 41 links, 40 joints
Joints:
- joint camera_fixed_joint: origin xyz=0.17 -0.03 0.05 rpy=0 1.578 0 -> xyz=0.0 0.17 0.05 rpy=-1.578 0 0

Commit message: Implement node to calculate IK using DH of the arm

File: src/quadruped_arm_motion/urdf/quadruped_arm_robot_control_real_effortTest_develope.urdf (robot description, URDF)
Before this commit: robot quadruped_arm_robot, 41 links, 40 joints
Joints:
- joint camera_fixed_joint: origin xyz=0.0 0.17 0.05 rpy=-1.578 0 0 -> xyz=0.17 0 0.0 rpy=-1.578 0 -1.578

Commit message: Is solve the IK is added joints of DH to test the DH on RVIZ is pending to solve the elbow problem

File: src/quadruped_arm_motion/urdf/quadruped_arm_robot_control_real_effortTest_develope.urdf (robot description, URDF)
Before this commit: robot quadruped_arm_robot, 41 links, 40 joints
Joints:
- joint camera_fixed_joint: origin xyz=0.17 0 0.0 rpy=-1.578 0 -1.578 -> xyz=0.25 0 0.0 rpy=-1.578 0 -1.578

Commit message: add ik solution into real robot

File: src/quadruped_arm_motion/urdf/quadruped_arm_robot_control_real_effortTest_develope.urdf (robot description, URDF)
Before this commit: robot quadruped_arm_robot, 41 links, 40 joints
Joints:
- joint camera_fixed_joint: origin xyz=0.25 0 0.0 rpy=-1.578 0 -1.578 -> xyz=0.25 0 0.0 rpy=-2.178 0 -1.578

Commit message: Fix DH an implement rotation parameter into IK

File: src/quadruped_arm_motion/urdf/quadruped_arm_robot_control_real_effortTest_develope.urdf (robot description, URDF)
Before this commit: robot quadruped_arm_robot, 41 links, 40 joints
Joints:
- joint camera_fixed_joint: origin xyz=0.25 0 0.0 rpy=-2.178 0 -1.578 -> xyz=0.01 0 0.0 rpy=-1.75 0 -1.578

Commit message: Fix Ik using peter corke toolbox and IKPy toolbox

File: src/quadruped_arm_motion/urdf/quadruped_arm_robot_control_real_effortTest_develope.urdf (robot description, URDF)
Before this commit: robot quadruped_arm_robot, 41 links, 40 joints
Joints:
- joint camera_fixed_joint: origin xyz=0.01 0 0.0 rpy=-1.75 0 -1.578 -> xyz=0.02 0 0.0 rpy=-1.75 0 -1.578
